Commit message: fix: added usds as instanceable meshes

File: objects_gazebo/bigbird/3m_high_tack_spray_adhesive/3m_high_tack_spray_adhesive.urdf (robot description, URDF)
Before this commit: robot 3m_high_tack_spray_adhesive, 1 links, 0 joints
Links:
- removed link 3m_high_tack_spray_adhesive__link
- added link base_link, mass 0.10653573521491269; collision mesh filename=./3m_high_tack_spray_adhesive_250_collision.obj scale=1.0 1.0 1.0; visual mesh filename=./optimized_tsdf_texture_mapped_mesh.obj scale=1.0 1.0 1.0

File: objects_gazebo/bigbird/advil_liqui_gels/advil_liqui_gels.urdf (robot description, URDF)
Before this commit: robot advil_liqui_gels, 1 links, 0 joints
Links:
- removed link advil_liqui_gels__link
- added link base_link, mass 0.030456724167062986; collision mesh filename=./advil_liqui_gels_250_collision.obj scale=1.0 1.0 1.0; visual mesh filename=./optimized_tsdf_texture_mapped_mesh.obj scale=1.0 1.0 1.0

File: objects_gazebo/bigbird/aunt_jemima_original_syrup/aunt_jemima_original_syrup.urdf (robot description, URDF)
Before this commit: robot aunt_jemima_original_syrup, 1 links, 0 joints
Links:
- removed link aunt_jemima_original_syrup__link
- added link base_link, mass 0.08773417526160335; collision mesh filename=./aunt_jemima_original_syrup_250_collision.obj scale=1.0 1.0 1.0; visual mesh filename=./optimized_tsdf_texture_mapped_mesh.obj scale=1.0 1.0 1.0

File: objects_gazebo/bigbird/bai5_sumatra_dragonfruit/bai5_sumatra_dragonfruit.urdf (robot description, URDF)
Before this commit: robot bai5_sumatra_dragonfruit, 1 links, 0 joints
Links:
- removed link bai5_sumatra_dragonfruit__link
- added link base_link, mass 0.06578220805355957; collision mesh filename=./bai5_sumatra_dragonfruit_250_collision.obj scale=1.0 1.0 1.0; visual mesh filename=./optimized_tsdf_texture_mapped_mesh.obj scale=1.0 1.0 1.0

File: objects_gazebo/bigbird/band_aid_clear_strips/band_aid_clear_strips.urdf (robot description, URDF)
Before this commit: robot band_aid_clear_strips, 1 links, 0 joints
Links:
- removed link band_aid_clear_strips__link
- added link base_link, mass 0.034060539105154275; collision mesh filename=./band_aid_clear_strips_250_collision.obj scale=1.0 1.0 1.0; visual mesh filename=./optimized_tsdf_texture_mapped_mesh.obj scale=1.0 1.0 1.0

File: objects_gazebo/bigbird/band_aid_sheer_strips/band_aid_sheer_strips.urdf (robot description, URDF)
Before this commit: robot band_aid_sheer_strips, 1 links, 0 joints
Links:
- removed link band_aid_sheer_strips__link
- added link base_link, mass 0.03946361469719523; collision mesh filename=./band_aid_sheer_strips_250_collision.obj scale=1.0 1.0 1.0; visual mesh filename=./optimized_tsdf_texture_mapped_mesh.obj scale=1.0 1.0 1.0

File: objects_gazebo/bigbird/blue_clover_baby_toy/blue_clover_baby_toy.urdf (robot description, URDF)
Before this commit: robot blue_clover_baby_toy, 1 links, 0 joints
Links:
- removed link blue_clover_baby_toy__link
- added link base_link, mass 0.0059535089510752166; collision mesh filename=./blue_clover_baby_toy_250_collision.obj scale=1.0 1.0 1.0; visual mesh filename=./optimized_tsdf_texture_mapped_mesh.obj scale=1.0 1.0 1.0

File: objects_gazebo/bigbird/bumblebee_albacore/bumblebee_albacore.urdf (robot description, URDF)
Before this commit: robot bumblebee_albacore, 1 links, 0 joints
Links:
- removed link bumblebee_albacore__link
- added link base_link, mass 0.01734206582504033; collision mesh filename=./bumblebee_albacore_250_collision.obj scale=1.0 1.0 1.0; visual mesh filename=./optimized_tsdf_texture_mapped_mesh.obj scale=1.0 1.0 1.0

File: objects_gazebo/bigbird/campbells_chicken_noodle_soup/campbells_chicken_noodle_soup.urdf (robot description, URDF)
Before this commit: robot campbells_chicken_noodle_soup, 1 links, 0 joints
Links:
- removed link campbells_chicken_noodle_soup__link
- added link base_link, mass 0.06058835323001838; collision mesh filename=./campbells_chicken_noodle_soup_250_collision.obj scale=1.0 1.0 1.0; visual mesh filename=./optimized_tsdf_texture_mapped_mesh.obj scale=1.0 1.0 1.0

File: objects_gazebo/bigbird/campbells_soup_at_hand_creamy_tomato/campbells_soup_at_hand_creamy_tomato.urdf (robot description, URDF)
Before this commit: robot campbells_soup_at_hand_creamy_tomato, 1 links, 0 joints
Links:
- removed link campbells_soup_at_hand_creamy_tomato__link
- added link base_link, mass 0.039711662220987716; collision mesh filename=./campbells_soup_at_hand_creamy_tomato_250_collision.obj scale=1.0 1.0 1.0; visual mesh filename=./optimized_tsdf_texture_mapped_mesh.obj scale=1.0 1.0 1.0

File: objects_gazebo/bigbird/canon_ack_e10_box/canon_ack_e10_box.urdf (robot description, URDF)
Before this commit: robot canon_ack_e10_box, 1 links, 0 joints
Links:
- removed link canon_ack_e10_box__link
- added link base_link, mass 0.09219330686975427; collision mesh filename=./canon_ack_e10_box_250_collision.obj scale=1.0 1.0 1.0; visual mesh filename=./optimized_tsdf_texture_mapped_mesh.obj scale=1.0 1.0 1.0

File: objects_gazebo/bigbird/cheez_it_white_cheddar/cheez_it_white_cheddar.urdf (robot description, URDF)
Before this commit: robot cheez_it_white_cheddar, 1 links, 0 joints
Links:
- removed link cheez_it_white_cheddar__link
- added link base_link, mass 0.1633816739891262; collision mesh filename=./cheez_it_white_cheddar_250_collision.obj scale=1.0 1.0 1.0; visual mesh filename=./optimized_tsdf_texture_mapped_mesh.obj scale=1.0 1.0 1.0

File: objects_gazebo/bigbird/chewy_dipps_chocolate_chip/chewy_dipps_chocolate_chip.urdf (robot description, URDF)
Before this commit: robot chewy_dipps_chocolate_chip, 1 links, 0 joints
Links:
- removed link chewy_dipps_chocolate_chip__link
- added link base_link, mass 0.10252997395123727; collision mesh filename=./chewy_dipps_chocolate_chip_250_collision.obj scale=1.0 1.0 1.0; visual mesh filename=./optimized_tsdf_texture_mapped_mesh.obj scale=1.0 1.0 1.0

File: objects_gazebo/bigbird/chewy_dipps_peanut_butter/chewy_dipps_peanut_butter.urdf (robot description, URDF)
Before this commit: robot chewy_dipps_peanut_butter, 1 links, 0 joints
Links:
- removed link chewy_dipps_peanut_butter__link
- added link base_link, mass 0.10357864080574644; collision mesh filename=./chewy_dipps_peanut_butter_250_collision.obj scale=1.0 1.0 1.0; visual mesh filename=./optimized_tsdf_texture_mapped_mesh.obj scale=1.0 1.0 1.0

File: objects_gazebo/bigbird/cholula_chipotle_hot_sauce/cholula_chipotle_hot_sauce.urdf (robot description, URDF)
Before this commit: robot cholula_chipotle_hot_sauce, 1 links, 0 joints
Links:
- removed link cholula_chipotle_hot_sauce__link
- added link base_link, mass 0.02623282392945838; collision mesh filename=./cholula_chipotle_hot_sauce_250_collision.obj scale=1.0 1.0 1.0; visual mesh filename=./optimized_tsdf_texture_mapped_mesh.obj scale=1.0 1.0 1.0

File: objects_gazebo/bigbird/cinnamon_toast_crunch/cinnamon_toast_crunch.urdf (robot description, URDF)
Before this commit: robot cinnamon_toast_crunch, 1 links, 0 joints
Links:
- removed link cinnamon_toast_crunch__link
- added link base_link, mass 0.310196837955065; collision mesh filename=./cinnamon_toast_crunch_250_collision.obj scale=1.0 1.0 1.0; visual mesh filename=./optimized_tsdf_texture_mapped_mesh.obj scale=1.0 1.0 1.0

File: objects_gazebo/bigbird/clif_crunch_chocolate_chip/clif_crunch_chocolate_chip.urdf (robot description, URDF)
Before this commit: robot clif_crunch_chocolate_chip, 1 links, 0 joints
Links:
- removed link clif_crunch_chocolate_chip__link
- added link base_link, mass 0.11995054073537159; collision mesh filename=./clif_crunch_chocolate_chip_250_collision.obj scale=1.0 1.0 1.0; visual mesh filename=./optimized_tsdf_texture_mapped_mesh.obj scale=1.0 1.0 1.0

File: objects_gazebo/bigbird/clif_crunch_peanut_butter/clif_crunch_peanut_butter.urdf (robot description, URDF)
Before this commit: robot clif_crunch_peanut_butter, 1 links, 0 joints
Links:
- removed link clif_crunch_peanut_butter__link
- added link base_link, mass 0.12031859818630702; collision mesh filename=./clif_crunch_peanut_butter_250_collision.obj scale=1.0 1.0 1.0; visual mesh filename=./optimized_tsdf_texture_mapped_mesh.obj scale=1.0 1.0 1.0

File: objects_gazebo/bigbird/clif_crunch_white_chocolate_macademia_nut/clif_crunch_white_chocolate_macademia_nut.urdf (robot description, URDF)
Before this commit: robot clif_crunch_white_chocolate_macademia_nut, 1 links, 0 joints
Links:
- removed link clif_crunch_white_chocolate_macademia_nut__link
- added link base_link, mass 0.12054650007775884; collision mesh filename=./clif_crunch_white_chocolate_macademia_nut_250_collision.o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 scale=1.0 1.0 1.0; visual mesh filename=./optimized_tsdf_texture_mapped_mesh.obj scale=1.0 1.0 1.0

File: objects_gazebo/bigbird/clif_z_bar_chocolate_chip/clif_z_bar_chocolate_chip.urdf (robot description, URDF)
Before this commit: robot clif_z_bar_chocolate_chip, 1 links, 0 joints
Links:
- removed link clif_z_bar_chocolate_chip__link
- added link base_link, mass 0.10548368926478464; collision mesh filename=./clif_z_bar_chocolate_chip_250_collision.obj scale=1.0 1.0 1.0; visual mesh filename=./optimized_tsdf_texture_mapped_mesh.obj scale=1.0 1.0 1.0
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